File: mains_io.kicad_sch (KiCad schematic)
At the start: 85 parts, among them J110 MAINS IN L/N, J111 K1 L/COM/NO, J112 K2 L/COM/NO, J113 K3 L/COM/NO, J114 K4 L/COM/NO, J115 END SW 1/2/3, J116 DEMAND 230V/24V/RET, K101 HF32FA-G/005-HSL1, K102 HF32FA-G/005-HSL1, K103 HF32FA-G/005-HSL1, K104 HF32FA-G/005-HSL1 (DNP), Q101 AO3400A, Q102 AO3400A, Q103 AO3400A, Q104 AO3400A, U101 LTV-817S, U102 LTV-817S, U103 LTV-817S, U104 LTV-817S, U105 LTV-817S

Commit message: Place and autoroute the board; add the reproducible routing pipeline
Board 150 x 95 mm, 2-layer, routed with Freerouting 2.5 from a placed
layout: DRC 0 violations / 0 unconnected, schematic parity clean, ERC clean.

- Isolation band, antenna keep-out, relay/opto slots, 6.4 mm mains-to-SELV
  custom DRC (heating-controller.kicad_dru) and MAINS / MAINS_SENSE / Power
  net classes in the project file.
- Fixed wiring laid before routing: L/N buses, relay COM/NO links,
  DEMAND_RET return, USB-C D+/D- bridges and VBUS escape, 31 GND stitching
  vias so the bottom pour stays in one piece.
- J115/J116 moved in from the board edge so every courtyard is inside the
  outline (JLC assembly margin).
- tools/route/: prep -> Freerouting -> SES import + pours -> DRC + gap fix,
  reproducible in ~2 min; outputs land in fab/route/ (ignored).
- Schematic: pin-type fixes in the project library, ESP32 thermal pads
  numbered; docs/design.md layout section rewritten to match the board.

Co-Authored-By: Claude Fable 5.1 <noreply@anthropic.com>
Connections:
- net S1_5 is gone; now on net S1_4: R118.2, R119.1
- net S2_5 is gone; now on net S2_4: R128.2, R129.1
- net S3_5 is gone; now on net S3_4: R138.2, R139.1
- net S5_5 is gone; now on net S5_4: R158.2, R159.1
- net DEMAND_24: now also D108.1 (K), R147.2, U104.1; no longer R148.2, R149.1
- net DEMAND_RET: now also R149.2; no longer D108.2 (A), U104.2
- net LEDA1: now also R116.2; no longer R119.2
- net LEDA2: now also R126.2; no longer R129.2
- net LEDA3: now also R136.2; no longer R139.2
- net LEDA5: now also R156.2; no longer R159.2
- net MAINS_N: now also R119.2, R129.2, R139.2, R159.2; no longer D105.2 (A), D106.2 (A), D107.2 (A), D109.2 (A), U101.2, U102.2, U103.2, U105.2
- net S1_3: now also R117.2, R118.1; no longer R116.2, R117.1
- net S1_4: no longer R117.2, R118.1
- net S2_3: now also R127.2, R128.1; no longer R126.2, R127.1
- net S2_4: no longer R127.2, R128.1
- net S3_3: now also R137.2, R138.1; no longer R136.2, R137.1
- net S3_4: no longer R137.2, R138.1
- net S4_4: now also R148.2, R149.1; no longer R147.2, R148.1
- net S5_3: now also R157.2, R158.1; no longer R156.2, R157.1
- net S5_4: no longer R157.2, R158.1
- removed net LEDA4: D108.1 (K), R149.2, U104.1
- new net LEDK1: D105.2 (A), R117.1, U101.2
- new net LEDK2: D106.2 (A), R127.1, U102.2
- new net LEDK3: D107.2 (A), R137.1, U103.2
- new net LEDK4: D108.2 (A), R148.1, U104.2
- new net LEDK5: D109.2 (A), R157.1, U105.2

Commit message: Address the independent design review: OT net split and fuse, 2.0 mm live-input class, demand detector margin, 3V3 copper, silkscreen
Two review rounds closed with design changes rather than prose:

- OpenTherm: U201 emitter and D207 cathode moved off OT_N1 onto OT_TXE
  (the net merge echoed our own TX into the RX opto); D208 SMAJ24A fitted;
  F201 1 A 250 V fast 2410 fuse in series with OT1 so a 230 V miswire is a
  calculable TVS-plus-fuse crowbar instead of parts failing open.
- Raw live inputs (ES1-3_IN, DEMAND_230) in a MAINS_IN class at 2.0 mm to
  everything, included in the 6.4 mm and edge rules; mains-to-mains 2.0 mm;
  the four inputs are pre-routed as locked lanes (the autorouter cannot
  thread them at that clearance); J115 wired ES3/ES2/ES1 top to bottom.
- Demand chain 3+3 and opto pull-ups 220 k after a time-domain model showed
  the 24 V detector had no margin; R15 330 R limits 1-Wire clamp current.
- +3V3 copper on the regulator tab (locked bars + pour, 125 mm2); GND island
  repair vias and stitching cleanup in the pipeline; silkscreen labels at
  every terminal pin plus warnings; LCSC/Description/Datasheet copied into
  the PCB footprints so schematic parity is clean (7 board-only items).
- Docs: design.md and requirements.md corrected where they had drifted;
  docs/layout-notes.md records what worked and failed in routing and margins.

Board: DRC 0 errors / 0 unconnected, ERC 0 errors, courtyards inside the
outline, Freerouting 40 passes in ~1 min.

Co-Authored-By: Claude Fable 5.1 <noreply@anthropic.com>
Claude-Session: https://claude.ai/code/session_01XDSh2Z4phxf7z2Gu1153CL
Parts:
- R110, R120, R130, R140, R150: value 47k -> 220k; LCSC C25819 -> C22961
Connections:
- net DEMAND_24: now also R146.2; no longer R147.2
- net ES1_IN: now also J115.3 (Pin_3); no longer J115.1 (Pin_1)
- net ES3_IN: now also J115.1 (Pin_1); no longer J115.3 (Pin_3)
- net LEDK4: now also R147.1; no longer R148.1
- net S4_3: now also R147.2, R148.1; no longer R146.2, R147.1
Changed lines of the file:
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@@
 			)
 		)
-		(property "Datasheet" "http://www.soselectronic.cz/a_info/resource/d/pc817.pdf"
+		(property "Datasheet" "https://www.lcsc.com/datasheet/lcsc_datasheet_2304140030_Lite-On-LTV-817S-TA1-C_C109227.pdf"
 			(at 62.23 224.79 0)
 			(hide yes)
@@
 			)
 		)
-		(property "Value" "47k"
+		(property "Value" "220k"
 			(at 82.55 204.47 90)
 			(effects
@@
 			)
 		)
-		(property "LCSC" "C25819"
+		(property "LCSC" "C22961"
 			(at 82.55 204.47 0)
 			(hide yes)
@@
 			)
 		)
-		(property "Datasheet" "http://www.soselectronic.cz/a_info/resource/d/pc817.pdf"
+		(property "Datasheet" "https://www.lcsc.com/datasheet/lcsc_datasheet_2304140030_Lite-On-LTV-817S-TA1-C_C109227.pdf"
 			(at 137.16 224.79 0)
 			(hide yes)
@@
 			)
 		)
-		(property "Value" "47k"
+		(property "Value" "220k"
 			(at 157.48 204.47 90)
 			(effects
@@
 			)
 		)
-		(property "LCSC" "C25819"
+		(property "LCSC" "C22961"
 			(at 157.48 204.47 0)
 			(hide yes)
@@
 			)
 		)
-		(property "Datasheet" "http://www.soselectronic.cz/a_info/resource/d/pc817.pdf"
+		(property "Datasheet" "https://www.lcsc.com/datasheet/lcsc_datasheet_2304140030_Lite-On-LTV-817S-TA1-C_C109227.pdf"
 			(at 212.09 224.79 0)
 			(hide yes)
@@
 			)
 		)
-		(property "Value" "47k"
+		(property "Value" "220k"
 			(at 232.41 204.47 90)
 			(effects
@@
 			)
 		)
-		(property "LCSC" "C25819"
+		(property "LCSC" "C22961"
 			(at 232.41 204.47 0)
 			(hide yes)
@@
 			)
 		)
-		(property "Datasheet" "http://www.soselectronic.cz/a_info/resource/d/pc817.pdf"
+		(property "Datasheet" "https://www.lcsc.com/datasheet/lcsc_datasheet_2304140030_Lite-On-LTV-817S-TA1-C_C109227.pdf"
 			(at 287.02 224.79 0)
 			(hide yes)
@@
 			)
 		)
-		(property "Value" "47k"
+		(property "Value" "220k"
 			(at 307.34 204.47 90)
 			(effects
@@
 			)
 		)
-		(property "LCSC" "C25819"
+		(property "LCSC" "C22961"
 			(at 307.34 204.47 0)
 			(hide yes)
@@
 			)
 		)
-		(property "Datasheet" "http://www.soselectronic.cz/a_info/resource/d/pc817.pdf"
+		(property "Datasheet" "https://www.lcsc.com/datasheet/lcsc_datasheet_2304140030_Lite-On-LTV-817S-TA1-C_C109227.pdf"
 			(at 361.95 224.79 0)
 			(hide yes)
@@
 			)
 		)
-		(property "Value" "47k"
+		(property "Value" "220k"
 			(at 382.27 204.47 90)
 			(effects
@@
 			)
 		)
-		(property "LCSC" "C25819"
+		(property "LCSC" "C22961"
 			(at 382.27 204.47 0)
 			(hide yes)
@@
 		)
 	)
-	(label "ES1_IN"
+	(label "ES3_IN"
 		(at 114.30 247.65 180)
 		(effects
@@
 		)
 	)
-	(label "ES3_IN"
+	(label "ES1_IN"
 		(at 114.30 252.73 180)
 		(effects
@@
 		)
 	)
-	(label "S4_3"
+	(label "DEMAND_24"
 		(at 255.27 184.15 270)
 		(effects
@@
 		)
 	)
-	(label "S4_3"
+	(label "LEDK4"
 		(at 255.27 186.69 90)
 		(effects
@@
 		)
 	)
-	(label "DEMAND_24"
+	(label "S4_3"
 		(at 255.27 194.31 270)
 		(effects
@@
 		)
 	)
-	(label "LEDK4"
+	(label "S4_3"
 		(at 255.27 195.58 90)
 		(effects

Commit message: Name the board Andiron v1.0; add BOM with cost estimates, renders, getting-started docs and CLAUDE.md
- Andiron v1.0 and the author name on the silkscreen, in every title block
  and in the README; J116 warning moved inside the board edge.
- tools/bom.py: BOM from the schematic with LCSC prices from the Konnect
  JLCPCB database -> docs/BOM.md (cost summary, Basic/Extended, DNP list) and
  docs/bom/andiron-bom-jlc.csv (JLCPCB upload). ~$15.77 components per board,
  ~$28.97 per board at 5 including assumed Extended-part fees.
- tools/sync_models.py relinks all 152 footprints to 3D models with portable
  ${KIPRJMOD} paths (also fixed in lib/jlc.pretty); stand-ins for the
  ESP32-C6 module and HRO USB-C. Wired into the routing pipeline.
- tools/render.sh: ray-traced 3D views and 2D layer plots in docs/images/.
- README rewritten: renders, BOM summary, getting started with Konnect MCP,
  repository layout. tools/README.md indexes every script; Konnect helpers
  and the pour-island check moved into tools/.
- CLAUDE.md: BOM and cost estimate kept current on every schematic change,
  definition of done for board changes.
- .konnect/project.json design rules brought in line with what is built;
  project-local .mcp.json for Konnect.
- Removed references to a commercial product; the docs now describe the
  board on its own terms, designed for Home Assistant and ESPHome.

ERC 0 errors; DRC 0 errors, 0 unconnected, parity clean.

Co-Authored-By: Claude Opus 5.5 <noreply@anthropic.com>
Claude-Session: https://claude.ai/code/session_01XDSh2Z4phxf7z2Gu1153CL
Other:
- company: (none) -> Cedric Van Goethem
- title: (none) -> Andiron
Changed lines of the file:
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@@
 	(generator_version "10.0")
 	(paper "A3")
+	(title_block
+		(title "Andiron")
+		(date "2026-10-22")
+		(rev "v1.0")
+		(company "Cedric Van Goethem")
+	)
   (text "MAINS IO. Relays K101-K104 switch MAINS_L to NO; link L-COM with a wire in the terminal for switched-live, or leave open for volt-free. K104 DNP. Gate pull-downs keep every relay OFF through reset/brownout."
     (at 30 30 0)
