File: relays.kicad_sch (KiCad schematic)
At the start: 32 parts, among them J111 K1 L/COM/NO, J112 K2 L/COM/NO, J113 K3 L/COM/NO, J114 K4 L/COM/NO, K101 HF115F/005-1ZS3A, K102 HF115F/005-1ZS3A, K103 HF115F/005-1ZS3A, K104 HF115F/005-1ZS3A, Q101 AO3400A, Q102 AO3400A, Q103 AO3400A, Q104 AO3400A

Commit message: Wall-hanging layout, cheaper parts, OLED area
Layout (160 x 95 mm): the board hangs on a wall with every cable from below
or the left. Relay and OpenTherm terminals on the bottom edge, USB-C, FLOW,
OUTDOOR and Qwiic on the left edge, antenna at the top edge. The OLED module
stacks in landscape over a reserved top-right area.

Parts: TE RT314005 relays replace the HF115F (same body and pin grid,
reinforced 5 kV / 10 mm insulation, flux-proof so no washing after THT); AEM
MF2410F1.000TM fast fuse replaces the Bourns (same breaking capacity and
I2t, Bourns nearly out of stock); Basic 100 nF and 1 uF capacitors.
Per-board total at 5: $37.23 -> $27.86 (components $24.03 -> $15.86).

Tooling: locked +5V rail and supply feed (Freerouting would not route the
net), USB-C pre-routes drawn in the receptacle's own frame, router keep-outs
over the isolation slots, temporary zones stripped in a text pass, wider
pour-island repair, a pre-routing placement check, and sanity checks for
connector edges, no-cable edges and the OLED area.

Co-Authored-By: Claude Opus 5.5 <noreply@anthropic.com>
Claude-Session: https://claude.ai/code/session_01XDSh2Z4phxf7z2Gu1153CL
Parts:
- J111: value K1 L/COM/NO -> CH1 NC/COM/NO
- J112: value K2 L/COM/NO -> CH2 NC/COM/NO
- J113: value K3 L/COM/NO -> CH3 NC/COM/NO
- J114: value K4 L/COM/NO -> CH4 NC/COM/NO
- K101, K102, K103, K104: value HF115F/005-1ZS3A -> RT314005; footprint jlc:RELAY-TH_HF115F-024-2ZS4 -> jlc:RELAY-TH_RT314005_HF115F-PINS; LCSC C882369 -> C7065270
Changed lines of the file:
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@@
 			)
 		)
-		(property "Value" "K1 L/COM/NO"
+		(property "Value" "CH1 NC/COM/NO"
 			(at 115.57 64.77 0)
 			(effects
@@
 			)
 		)
-		(property "Value" "K2 L/COM/NO"
+		(property "Value" "CH2 NC/COM/NO"
 			(at 209.55 64.77 0)
 			(effects
@@
 			)
 		)
-		(property "Value" "K3 L/COM/NO"
+		(property "Value" "CH3 NC/COM/NO"
 			(at 304.8 64.77 0)
 			(effects
@@
 			)
 		)
-		(property "Value" "K4 L/COM/NO"
+		(property "Value" "CH4 NC/COM/NO"
 			(at 400.05 64.77 0)
 			(effects
@@
 			)
 		)
-		(property "Value" "HF115F/005-1ZS3A"
+		(property "Value" "RT314005"
 			(at 69.85 55.88 0)
 			(effects
@@
 			)
 		)
-		(property "Footprint" "jlc:RELAY-TH_HF115F-024-2ZS4"
+		(property "Footprint" "jlc:RELAY-TH_RT314005_HF115F-PINS"
 			(at 69.85 40.64 0)
 			(hide yes)
@@
 			)
 		)
-		(property "Datasheet" "https://www.lcsc.com/datasheet/C882369.pdf"
+		(property "Datasheet" "https://www.lcsc.com/datasheet/lcsc_datasheet_2404231543_TE-Connectivity-RT314005_C7065270.pdf"
 			(at 69.85 40.64 0)
 			(hide yes)
@@
 			)
 		)
-		(property "LCSC" "C882369"
+		(property "LCSC" "C7065270"
 			(at 69.85 40.64 0)
 			(hide yes)
@@
 			)
 		)
-		(property "Value" "HF115F/005-1ZS3A"
+		(property "Value" "RT314005"
 			(at 165.1 55.88 0)
 			(effects
@@
 			)
 		)
-		(property "Footprint" "jlc:RELAY-TH_HF115F-024-2ZS4"
+		(property "Footprint" "jlc:RELAY-TH_RT314005_HF115F-PINS"
 			(at 165.1 40.64 0)
 			(hide yes)
@@
 			)
 		)
-		(property "Datasheet" "https://www.lcsc.com/datasheet/C882369.pdf"
+		(property "Datasheet" "https://www.lcsc.com/datasheet/lcsc_datasheet_2404231543_TE-Connectivity-RT314005_C7065270.pdf"
 			(at 165.1 40.64 0)
 			(hide yes)
@@
 			)
 		)
-		(property "LCSC" "C882369"
+		(property "LCSC" "C7065270"
 			(at 165.1 40.64 0)
 			(hide yes)
@@
 			)
 		)
-		(property "Value" "HF115F/005-1ZS3A"
+		(property "Value" "RT314005"
 			(at 260.35 55.88 0)
 			(effects
@@
 			)
 		)
-		(property "Footprint" "jlc:RELAY-TH_HF115F-024-2ZS4"
+		(property "Footprint" "jlc:RELAY-TH_RT314005_HF115F-PINS"
 			(at 260.35 40.64 0)
 			(hide yes)
@@
 			)
 		)
-		(property "Datasheet" "https://www.lcsc.com/datasheet/C882369.pdf"
+		(property "Datasheet" "https://www.lcsc.com/datasheet/lcsc_datasheet_2404231543_TE-Connectivity-RT314005_C7065270.pdf"
 			(at 260.35 40.64 0)
 			(hide yes)
@@
 			)
 		)
-		(property "LCSC" "C882369"
+		(property "LCSC" "C7065270"
 			(at 260.35 40.64 0)
 			(hide yes)
@@
 			)
 		)
-		(property "Value" "HF115F/005-1ZS3A"
+		(property "Value" "RT314005"
 			(at 355.6 55.88 0)
 			(effects
@@
 			)
 		)
-		(property "Footprint" "jlc:RELAY-TH_HF115F-024-2ZS4"
+		(property "Footprint" "jlc:RELAY-TH_RT314005_HF115F-PINS"
 			(at 355.6 40.64 0)
 			(hide yes)
@@
 			)
 		)
-		(property "Datasheet" "https://www.lcsc.com/datasheet/C882369.pdf"
+		(property "Datasheet" "https://www.lcsc.com/datasheet/lcsc_datasheet_2404231543_TE-Connectivity-RT314005_C7065270.pdf"
 			(at 355.6 40.64 0)
 			(hide yes)
@@
 			)
 		)
-		(property "LCSC" "C882369"
+		(property "LCSC" "C7065270"
 			(at 355.6 40.64 0)
 			(hide yes)
