File: opentherm.kicad_sch (KiCad schematic)
At the start: 17 parts, among them J201 OT (24V max), Q201 S8550, U201 LTV-817S (TX), U202 LTV-817S (RX)

Commit message: Address the independent design review: OT net split and fuse, 2.0 mm live-input class, demand detector margin, 3V3 copper, silkscreen
Two review rounds closed with design changes rather than prose:

- OpenTherm: U201 emitter and D207 cathode moved off OT_N1 onto OT_TXE
  (the net merge echoed our own TX into the RX opto); D208 SMAJ24A fitted;
  F201 1 A 250 V fast 2410 fuse in series with OT1 so a 230 V miswire is a
  calculable TVS-plus-fuse crowbar instead of parts failing open.
- Raw live inputs (ES1-3_IN, DEMAND_230) in a MAINS_IN class at 2.0 mm to
  everything, included in the 6.4 mm and edge rules; mains-to-mains 2.0 mm;
  the four inputs are pre-routed as locked lanes (the autorouter cannot
  thread them at that clearance); J115 wired ES3/ES2/ES1 top to bottom.
- Demand chain 3+3 and opto pull-ups 220 k after a time-domain model showed
  the 24 V detector had no margin; R15 330 R limits 1-Wire clamp current.
- +3V3 copper on the regulator tab (locked bars + pour, 125 mm2); GND island
  repair vias and stitching cleanup in the pipeline; silkscreen labels at
  every terminal pin plus warnings; LCSC/Description/Datasheet copied into
  the PCB footprints so schematic parity is clean (7 board-only items).
- Docs: design.md and requirements.md corrected where they had drifted;
  docs/layout-notes.md records what worked and failed in routing and margins.

Board: DRC 0 errors / 0 unconnected, ERC 0 errors, courtyards inside the
outline, Freerouting 40 passes in ~1 min.

Co-Authored-By: Claude Fable 5.1 <noreply@anthropic.com>
Claude-Session: https://claude.ai/code/session_01XDSh2Z4phxf7z2Gu1153CL
Parts:
- added F201: 1A 250V fast, Fuse:Fuse_Littelfuse-NANO2-451_453, symbol Device:Fuse
- D208: value SMAJ24A (DNP) -> SMAJ24A; now fitted
Connections:
- net OT1: now also F201.2; no longer J201.1 (Pin_1)
- net OT_N1: no longer D207.1 (K), U201.3
- new net OT1_IN: F201.1, J201.1 (Pin_1)
- new net OT_TXE: D207.1 (K), U201.3

Commit message: Name the board Andiron v1.0; add BOM with cost estimates, renders, getting-started docs and CLAUDE.md
- Andiron v1.0 and the author name on the silkscreen, in every title block
  and in the README; J116 warning moved inside the board edge.
- tools/bom.py: BOM from the schematic with LCSC prices from the Konnect
  JLCPCB database -> docs/BOM.md (cost summary, Basic/Extended, DNP list) and
  docs/bom/andiron-bom-jlc.csv (JLCPCB upload). ~$15.77 components per board,
  ~$28.97 per board at 5 including assumed Extended-part fees.
- tools/sync_models.py relinks all 152 footprints to 3D models with portable
  ${KIPRJMOD} paths (also fixed in lib/jlc.pretty); stand-ins for the
  ESP32-C6 module and HRO USB-C. Wired into the routing pipeline.
- tools/render.sh: ray-traced 3D views and 2D layer plots in docs/images/.
- README rewritten: renders, BOM summary, getting started with Konnect MCP,
  repository layout. tools/README.md indexes every script; Konnect helpers
  and the pour-island check moved into tools/.
- CLAUDE.md: BOM and cost estimate kept current on every schematic change,
  definition of done for board changes.
- .konnect/project.json design rules brought in line with what is built;
  project-local .mcp.json for Konnect.
- Removed references to a commercial product; the docs now describe the
  board on its own terms, designed for Home Assistant and ESPHome.

ERC 0 errors; DRC 0 errors, 0 unconnected, parity clean.

Co-Authored-By: Claude Opus 5.5 <noreply@anthropic.com>
Claude-Session: https://claude.ai/code/session_01XDSh2Z4phxf7z2Gu1153CL
Other:
- company: (none) -> Cedric Van Goethem
- title: (none) -> Andiron
Changed lines of the file:
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@@
 	(generator_version "10.0")
 	(paper "A4")
+	(title_block
+		(title "Andiron")
+		(date "2026-10-22")
+		(rev "v1.0")
+		(company "Cedric Van Goethem")
+	)
 	(text "OPENTHERM MASTER ADAPTER (Ihor Melnyk topology). Bus is boiler-powered SELV, polarity independent. OT_OUT high -> U201 on -> extra bus current (TX). Boiler voltage high -> D206 conducts -> Q201 on -> U202 on -> OT_IN high (RX). D208 TVS is DNP."
 		(at 20 30 0)

Commit message: Wall-hanging layout, cheaper parts, OLED area
Layout (160 x 95 mm): the board hangs on a wall with every cable from below
or the left. Relay and OpenTherm terminals on the bottom edge, USB-C, FLOW,
OUTDOOR and Qwiic on the left edge, antenna at the top edge. The OLED module
stacks in landscape over a reserved top-right area.

Parts: TE RT314005 relays replace the HF115F (same body and pin grid,
reinforced 5 kV / 10 mm insulation, flux-proof so no washing after THT); AEM
MF2410F1.000TM fast fuse replaces the Bourns (same breaking capacity and
I2t, Bourns nearly out of stock); Basic 100 nF and 1 uF capacitors.
Per-board total at 5: $37.23 -> $27.86 (components $24.03 -> $15.86).

Tooling: locked +5V rail and supply feed (Freerouting would not route the
net), USB-C pre-routes drawn in the receptacle's own frame, router keep-outs
over the isolation slots, temporary zones stripped in a text pass, wider
pour-island repair, a pre-routing placement check, and sanity checks for
connector edges, no-cable edges and the OLED area.

Co-Authored-By: Claude Opus 5.5 <noreply@anthropic.com>
Claude-Session: https://claude.ai/code/session_01XDSh2Z4phxf7z2Gu1153CL
Parts:
- F201: LCSC C1236062 -> C83798
Changed lines of the file:
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@@
 			)
 		)
-		(property "Datasheet" "https://wmsc.lcsc.com/wmsc/upload/file/pdf/v2/lcsc/2401290932_BOURNS-SF-2410FPA100W-2_C1236062.pdf"
+		(property "Datasheet" "https://www.lcsc.com/datasheet/lcsc_datasheet_2009081106_AEM-MF2410F1-000TM_C83798.pdf"
 			(at 26.67 88.9 0)
 			(hide yes)
@@
 			)
 		)
-		(property "LCSC" "C1236062"
+		(property "LCSC" "C83798"
 			(at 26.67 88.9 0)
 			(hide yes)

Commit message: JLC package, placement corrections, Preferred-part swaps
- tools/fab.sh builds the JLCPCB package in fab/jlc/: Gerbers and drill
  zip, BOM copy and a placement file from tools/cpl.py.
- tools/cpl.py applies JLC's orientation conventions per footprint
  (SOT-23/SOT-223 180°, SOT-23-6 -90°, pin headers 90° at the pad centre,
  USB-C at the pad centre), each checked in JLC's placement viewer.
- D1/D2 (SMF5.0A), D208 (SMAJ24A) and D205-D207 (BZT52) moved to the same
  part types from JLC's Preferred library: no Extended-part fee on Economic
  assembly. Datasheets checked; footprints unchanged, no rerouting.
- TVS descriptions corrected to unidirectional.
- bom.py no longer charges the fee on Preferred parts.
- Cost at 5 boards incl. fees: $27.86 -> $24.79 per board estimate; JLC
  quote for 2 assembled boards $104.09 -> $87.98.
- Renders and schematic PDF regenerated; JLC upload lessons in
  layout-notes.

Co-Authored-By: Claude Opus 5.5 <noreply@anthropic.com>
Claude-Session: https://claude.ai/code/session_01XDSh2Z4phxf7z2Gu1153CL
Parts:
- D205: LCSC C2116 -> C19077400
- D206: LCSC C2104 -> C19077412
- D207: LCSC C2115 -> C19077399
- D208: LCSC C89612 -> C19077541
Changed lines of the file:
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@@
 			)
 		)
-		(property "LCSC" "C2116"
+		(property "LCSC" "C19077400"
 			(at 139.7 110.49 0)
 			(hide yes)
@@
 			)
 		)
-		(property "LCSC" "C2104"
+		(property "LCSC" "C19077412"
 			(at 160.02 100.33 0)
 			(hide yes)
@@
 			)
 		)
-		(property "LCSC" "C2115"
+		(property "LCSC" "C19077399"
 			(at 175.26 129.54 0)
 			(hide yes)
@@
 			)
 		)
-		(property "Description" "Bidirectional transient-voltage-suppression diode"
+		(property "Description" "Unidirectional transient-voltage-suppression diode, cathode (pin 1) on the protected rail"
 			(at 100.33 154.94 0)
 			(hide yes)
@@
 			)
 		)
-		(property "LCSC" "C89612"
+		(property "LCSC" "C19077541"
 			(at 100.33 154.94 0)
 			(hide yes)
